Commit message: tuned PID gripper

File: src/armpi_gazebo/urdf/gazebo_armpi_fpv_edit.urdf (robot description, URDF)
Before this commit: robot armpi_fpv, 16 links, 15 joints
Joints:
- joint r_joint: limit lower=-2.57 upper=1.57 effort=20 velocity=5 -> lower=-2.57 upper=1.00 effort=20 velocity=5

Commit message: gripper control and spawn cube

File: src/armpi_gazebo/urdf/gazebo_armpi_fpv_edit.urdf (robot description, URDF)
Before this commit: robot armpi_fpv, 16 links, 15 joints
Joints:
- joint r_joint: limit lower=-2.57 upper=1.00 effort=20 velocity=5 -> lower=-2.57 upper=1.57 effort=20 velocity=5
